Commit message: bigman only legs

File: app/robots/bigman_only_legs/bigman_torqueBalancing_only_legs.urdf (robot description, URDF)
Before this commit: robot bigman, 53 links, 52 joints
Links:
- removed link DWL
- removed link DWS
- removed link DWYTorso
- removed link NeckPitch
- removed link NeckYaw
- removed link TorsoProtections
- removed link backpack
- removed link gaze
- removed link multisense/center_bottom_led_frame
- removed link multisense/center_top_led_frame
- removed link multisense/head
- removed link multisense/head_hokuyo_frame
- removed link multisense/head_imu_link
- removed link multisense/hokuyo_link
- removed link multisense/left_camera_frame
- removed link multisense/left_camera_optical_frame
- removed link multisense/left_led_frame
- removed link multisense/right_camera_frame
- removed link multisense/right_camera_optical_frame
- removed link multisense/right_led_frame
- removed link torso
- added link ExtraWeight, mass 20.0; collision cylinder length=0.15 radius=0.14; visual cylinder length=0.15 radius=0.14
- added link PelvisWeightBench, mass 5.5278386; collision mesh filename=package://bigman_urdf/meshes/simple/PelvisWeightBench.STL scale=0.001 0.001 0.001; visual mesh filename=package://bigman_urdf/meshes/PelvisWeightBench.STL scale=0.001 0.001 0.001
- link l_sole: mass 0 -> None
- link r_sole: mass 0 -> None
Joints:
- removed joint NeckPitchj
- removed joint NeckYawj
- removed joint WaistLat
- removed joint WaistSag
- removed joint WaistYaw
- removed joint backpack_joint
- removed joint center_bottom_led_frame_joint
- removed joint center_top_led_frame_joint
- removed joint gaze_joint
- removed joint head_hokuyo_joint
- removed joint head_imu_joint
- removed joint hokuyo_joint
- removed joint left_camera_frame_joint
- removed joint left_camera_optical_frame_joint
- removed joint left_led_frame_joint
- removed joint neck_joint
- removed joint right_camera_frame_joint
- removed joint right_camera_optical_frame_joint
- removed joint right_led_frame_joint
- removed joint torso_joint
- removed joint torso_protection_joint
- added joint ExtraWeight_joint: type fixed, parent PelvisWeightBench, child ExtraWeight, origin xyz=0.0 0 0.39 rpy=0 0 0
- added joint PelvisWeightBench_joint: type fixed, parent Waist, child PelvisWeightBench, origin xyz=-0.035 0 0.075 rpy=0 0 1.57079632679
