Commit message: added the contact frames at the legs

File: app/robots/icubGazeboSim/model.urdf (robot description, URDF)
Before this commit: robot iCub, 56 links, 55 joints
Links:
- added link l_upper_leg_contact, mass 0
- added link r_upper_leg_contact, mass 0
Joints:
- added joint l_upper_leg_frame_fixed_joint: type fixed, parent l_upper_leg, child l_upper_leg_contact, origin xyz=-0.0596 -0.0700 -0.0009 rpy=-1.5810 -0.2157 -1.5231, axis 0 0 0
- added joint r_upper_leg_frame_fixed_joint: type fixed, parent r_upper_leg, child r_upper_leg_contact, origin xyz=-0.0596 -0.0694 -0.0008 rpy=-1.5606 0.2124 -1.5229, axis 0 0 0
